Commit message: 解决冲突

File: franka/franka.urdf (robot description, URDF)
Before this commit: robot panda, 13 links, 12 joints
Links:
- link panda_hand: geometry collision mesh filename=./franka_description/meshes/collision/hand.stl; visual mesh filename=./franka_description/meshes/visual/hand.dae
- link panda_leftfinger: geometry collision mesh filename=./franka_description/meshes/collision/finger.stl; visual mesh filename=./franka_description/meshes/visual/finger.dae
- link panda_link0: geometry collision mesh filename=./franka_description/meshes/collision/link0.stl; visual mesh filename=./franka_description/meshes/visual/link0.dae
- link panda_link1: geometry collision mesh filename=./franka_description/meshes/collision/link1.stl; visual mesh filename=./franka_description/meshes/visual/link1.dae
- link panda_link2: geometry collision mesh filename=./franka_description/meshes/collision/link2.stl; visual mesh filename=./franka_description/meshes/visual/link2.dae
- link panda_link3: geometry collision mesh filename=./franka_description/meshes/collision/link3.stl; visual mesh filename=./franka_description/meshes/visual/link3.dae
- link panda_link4: geometry collision mesh filename=./franka_description/meshes/collision/link4.stl; visual mesh filename=./franka_description/meshes/visual/link4.dae
- link panda_link5: geometry collision mesh filename=./franka_description/meshes/collision/link5.stl; visual mesh filename=./franka_description/meshes/visual/link5.dae
- link panda_link6: geometry collision mesh filename=./franka_description/meshes/collision/link6.stl; visual mesh filename=./franka_description/meshes/visual/link6.dae
- link panda_link7: geometry collision mesh filename=./franka_description/meshes/collision/link7.stl; visual mesh filename=./franka_description/meshes/visual/link7.dae
- link panda_rightfinger: geometry collision mesh filename=./franka_description/meshes/collision/finger.stl; visual mesh filename=./franka_description/meshes/visual/finger.dae

File: iiwa/iiwa.urdf (robot description, URDF)
Before this commit: robot iiwa14, 10 links, 9 joints
Links:
- link iiwa_link_0: geometry collision box size=0.24 0.23 0.1575; visual mesh filename=./iiwa_description/meshes/link_0.stl
- link iiwa_link_1: geometry collision box size=0.175 0.19 0.26; visual mesh filename=./iiwa_description/meshes/link_1.stl
- link iiwa_link_2: geometry collision box size=0.175 0.24 0.19; visual mesh filename=./iiwa_description/meshes/link_2.stl
- link iiwa_link_3: geometry collision box size=0.125 0.15 0.26; visual mesh filename=./iiwa_description/meshes/link_3.stl
- link iiwa_link_4: geometry collision box size=0.125 0.22 0.15; visual mesh filename=./iiwa_description/meshes/link_4.stl
- link iiwa_link_5: geometry collision box size=0.125 0.15 0.24; visual mesh filename=./iiwa_description/meshes/link_5.stl
- link iiwa_link_6: geometry collision box size=0.125 0.15 0.125; visual mesh filename=./iiwa_description/meshes/link_6.stl
- link iiwa_link_7: geometry collision box size=0.1 0.1 0.05; visual mesh filename=./iiwa_description/meshes/link_7.stl

File: ur3e/ur3e.urdf (robot description, URDF)
Before this commit: robot ur3e_with_schunk_hand, 11 links, 10 joints
Links:
- link base_link_inertia: geometry collision mesh filename=./ur3e_description/meshes/ur3e/collision/base.stl; visual mesh filename=./ur3e_description/meshes/ur3e/visual/base.dae
- link forearm_link: geometry collision mesh filename=./ur3e_description/meshes/ur3e/collision/forearm.stl; visual mesh filename=./ur3e_description/meshes/ur3e/visual/forearm.dae
- link shoulder_link: geometry collision mesh filename=./ur3e_description/meshes/ur3e/collision/shoulder.stl; visual mesh filename=./ur3e_description/meshes/ur3e/visual/shoulder.dae
- link upper_arm_link: geometry collision mesh filename=./ur3e_description/meshes/ur3e/collision/upperarm.stl; visual mesh filename=./ur3e_description/meshes/ur3e/visual/upperarm.dae
- link wrist_1_link: geometry collision mesh filename=./ur3e_description/meshes/ur3e/collision/wrist1.stl; visual mesh filename=./ur3e_description/meshes/ur3e/visual/wrist1.dae
- link wrist_2_link: geometry collision mesh filename=./ur3e_description/meshes/ur3e/collision/wrist2.stl; visual mesh filename=./ur3e_description/meshes/ur3e/visual/wrist2.dae
- link wrist_3_link: geometry collision mesh filename=./ur3e_description/meshes/ur3e/collision/wrist3.stl; visual mesh filename=./ur3e_description/meshes/ur3e/visual/wrist3.dae
