Commit message: Your commit message

File: models/ur3e/ur3e_with_schunk_hand.urdf (robot description, URDF)
Before this commit: robot ur3e_with_schunk_hand, 42 links, 41 joints
Links:
- link base_link_inertia: geometry collision mesh filename=ur3e_description/meshes/ur3e/collision/base.stl; visual mesh filename=ur3e_description/meshes/ur3e/visual/base.dae
- link forearm_link: geometry collision mesh filename=ur3e_description/meshes/ur3e/collision/forearm.stl; visual mesh filename=ur3e_description/meshes/ur3e/visual/forearm.dae
- link right_hand_a: geometry collision mesh filename=ur3e_description/meshes/schunk_hand/d11.dae scale=1 1 1; visual mesh filename=ur3e_description/meshes/schunk_hand/d11.dae scale=1 1 1
- link right_hand_b: geometry collision mesh filename=ur3e_description/meshes/schunk_hand/d12.dae scale=1 1 1; visual mesh filename=ur3e_description/meshes/schunk_hand/d12.dae scale=1 1 1
- link right_hand_base_link: geometry collision mesh filename=ur3e_description/meshes/schunk_hand/base10.dae; visual mesh filename=ur3e_description/meshes/schunk_hand/base10.dae
- link right_hand_c: geometry collision mesh filename=ur3e_description/meshes/schunk_hand/d13.dae scale=1 1 1; visual mesh filename=ur3e_description/meshes/schunk_hand/d13.dae scale=1 1 1
- link right_hand_e1: geometry collision mesh filename=ur3e_description/meshes/schunk_hand/h10.dae scale=1 1 1; visual mesh filename=ur3e_description/meshes/schunk_hand/h10.dae scale=1 1 1
- link right_hand_e2: geometry collision mesh filename=ur3e_description/meshes/schunk_hand/h11.dae scale=1 1 1; visual mesh filename=ur3e_description/meshes/schunk_hand/h11.dae scale=1 1 1
- link right_hand_i: geometry collision mesh filename=ur3e_description/meshes/schunk_hand/f41.dae; visual mesh filename=ur3e_description/meshes/schunk_hand/f41.dae
- link right_hand_j: geometry collision mesh filename=ur3e_description/meshes/schunk_hand/f31.dae; visual mesh filename=ur3e_description/meshes/schunk_hand/f31.dae
- link right_hand_k: geometry collision mesh filename=ur3e_description/meshes/schunk_hand/f21.dae; visual mesh filename=ur3e_description/meshes/schunk_hand/f21.dae
- link right_hand_l: geometry collision mesh filename=ur3e_description/meshes/schunk_hand/f11.dae; visual mesh filename=ur3e_description/meshes/schunk_hand/f11.dae
- link right_hand_m: geometry collision mesh filename=ur3e_description/meshes/schunk_hand/f42.dae; visual mesh filename=ur3e_description/meshes/schunk_hand/f42.dae
- link right_hand_n: geometry collision mesh filename=ur3e_description/meshes/schunk_hand/f32.dae; visual mesh filename=ur3e_description/meshes/schunk_hand/f32.dae
- link right_hand_o: geometry collision mesh filename=ur3e_description/meshes/schunk_hand/f22.dae; visual mesh filename=ur3e_description/meshes/schunk_hand/f22.dae
- link right_hand_p: geometry collision mesh filename=ur3e_description/meshes/schunk_hand/f12.dae; visual mesh filename=ur3e_description/meshes/schunk_hand/f12.dae
- link right_hand_q: geometry collision mesh filename=ur3e_description/meshes/schunk_hand/f43.dae; visual mesh filename=ur3e_description/meshes/schunk_hand/f43.dae
- link right_hand_r: geometry collision mesh filename=ur3e_description/meshes/schunk_hand/f33.dae; visual mesh filename=ur3e_description/meshes/schunk_hand/f33.dae
- link right_hand_s: geometry collision mesh filename=ur3e_description/meshes/schunk_hand/f23.dae; visual mesh filename=ur3e_description/meshes/schunk_hand/f23.dae
- link right_hand_t: geometry collision mesh filename=ur3e_description/meshes/schunk_hand/f13.dae; visual mesh filename=ur3e_description/meshes/schunk_hand/f13.dae
- link right_hand_virtual_i: geometry collision mesh filename=ur3e_description/meshes/schunk_hand/f40.dae; visual mesh filename=ur3e_description/meshes/schunk_hand/f40.dae
- link right_hand_virtual_j: geometry collision mesh filename=ur3e_description/meshes/schunk_hand/f30.dae; visual mesh filename=ur3e_description/meshes/schunk_hand/f30.dae
- link right_hand_virtual_k: geometry collision mesh filename=ur3e_description/meshes/schunk_hand/f20.dae; visual mesh filename=ur3e_description/meshes/schunk_hand/f20.dae
- link right_hand_virtual_l: geometry collision mesh filename=ur3e_description/meshes/schunk_hand/f10.dae; visual mesh filename=ur3e_description/meshes/schunk_hand/f10.dae
- link right_hand_z: geometry collision mesh filename=ur3e_description/meshes/schunk_hand/d10.dae scale=1 1 1; visual mesh filename=ur3e_description/meshes/schunk_hand/d10.dae scale=1 1 1
- link shoulder_link: geometry collision mesh filename=ur3e_description/meshes/ur3e/collision/shoulder.stl; visual mesh filename=ur3e_description/meshes/ur3e/visual/shoulder.dae
- link upper_arm_link: geometry collision mesh filename=ur3e_description/meshes/ur3e/collision/upperarm.stl; visual mesh filename=ur3e_description/meshes/ur3e/visual/upperarm.dae
- link wrist_1_link: geometry collision mesh filename=ur3e_description/meshes/ur3e/collision/wrist1.stl; visual mesh filename=ur3e_description/meshes/ur3e/visual/wrist1.dae
- link wrist_2_link: geometry collision mesh filename=ur3e_description/meshes/ur3e/collision/wrist2.stl; visual mesh filename=ur3e_description/meshes/ur3e/visual/wrist2.dae
- link wrist_3_link: geometry collision mesh filename=ur3e_description/meshes/ur3e/collision/wrist3.stl; visual mesh filename=ur3e_description/meshes/ur3e/visual/wrist3.dae
